Commit message: Standardize TF base_link frame as boat to match localization

File: src/sailbot_sim/urdf/boat.urdf (robot description, URDF)
Before this commit: robot sailbot, 2 links, 1 joints
Links:
- removed link base_link
- added link boat; visual box size=0.5 0.2 0.2
Joints:
- joint base_to_sail: parent base_link -> boat
